File: Hardware/mppt/mppt.sch (EAGLE design)
At the start: 37 parts, among them M1 IRLZ34N, M2 IRLZ34N, M3 IRLZ34N

Commit message: Added lates MPPT Tracking PCB design
Also cleaned hardware folder, removing non-working current sense
designs.
Parts:
- removed C3: 100uF, capacitor-wima:C2.5/2
- removed C9: 1uF, capacitor-wima:C2.5/2
- removed D3: UF4007, diode:1N4004
- removed J5: (no value), con-lstb:MA05-1
- removed M1, M2, M3: IRLZ34N, transistor-power:PMOSFET_NTO220BV
- added D4: US1D - 1625280, diode:DIODE-DO-214AC
- added EN: (no value), jumper:SJ
- added INPUTS, OUTPUTS: (no value), con-lstb:MA05-1
- added U1, U2, U3: DMS3016SSS-13, equinox:DMS3016SSS-13
- BATT, SOL: value (none) -> TERMINAL_2WAY; device con-wago-508:W237-02P -> equinox:TERMINAL_2WAY
- C10, C11, C2, C5: device capacitor-wima:C2.5/2 -> resistor:C-EUC0805K
- C4: device capacitor-wima:C2.5/2 -> resistor:C-EU025-050X050
- C6: value 100uF -> 220uF; device capacitor-wima:C2.5/2 -> resistor:C-EU025-050X050
- C7, C8: value 1uF -> 0.1uF; device capacitor-wima:C2.5/2 -> resistor:C-EUC0805K
- D1, D2: value 1N4001 -> S1A-E3/5AT; device diode:1N4148 -> diode:DIODE-DO-214AC
- RSENSE2, RSENSE_BATT: device rcl:R-EU_R2512W -> rcl:R-EU_R2512
Connections:
- removed net BATT_AMPS: R_GAIN1.2, SENSE_AMP_BATT.OUT
- removed net BAT_VOLTS: C8.2, R5.1, R6.2
- removed net SOL_AMPS: R_GAIN.2, SENSE_AMP_SOL.OUT
- removed net SOL_VOLTS: C7.2, R3.1, R4.2
- new net BATT_I: OUTPUTS.4, R_GAIN1.2, SENSE_AMP_BATT.OUT
- new net BATT_V: C8.2, OUTPUTS.5, R5.1, R6.2
- new net SOL_I: OUTPUTS.2, R_GAIN.2, SENSE_AMP_SOL.OUT
- new net SOL_V: C7.2, OUTPUTS.3, R3.1, R4.2
- net EN_: now also EN.2, INPUTS.4; no longer J5.4
- net GND: now also BATT.P$2, D4.A, EN.1, INPUTS.1, INPUTS.2, INPUTS.3, OUTPUTS.1, SOL.P$2, U3.S, U3.S_2, U3.S_3; no longer BATT-1.KL, C3.1, C9.2, D3.A, M3.S, SOL-2.KL
- net N$11: now also R10.1, U3.G; no longer C2.2, C5.1, D3.C, GATE_DRIVE.VS, M2.S, M3.D, U$1.P$1
- net N$12: no longer C9.1
- net N$14: now also U2.G; no longer M2.G
- net N$16: now also SOL.P$1; no longer SOL-1.KL
- net N$3: now also BATT.P$1; no longer BATT-2.KL
- net N$4: now also C2.2, C5.1, D4.C, GATE_DRIVE.VS, U$1.P$1, U2.S, U2.S_2, U2.S_3, U3.D, U3.D_2, U3.D_3, U3.D_4; no longer M3.G, R10.1
- net N$5: now also U1.G; no longer M1.G
- net N$6: now also U1.D, U1.D_2, U1.D_3, U1.D_4, U2.D, U2.D_2, U2.D_3, U2.D_4; no longer M1.D, M2.D
- net N$9: now also U1.S, U1.S_2, U1.S_3; no longer C3.2, M1.S
- net PWM: now also INPUTS.5; no longer J5.5
Other:
- moved on the sheet: C11, C2, C5, C6, C8, D1, D2, GATE_DRIVE, R1, R10, R2, R5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

Commit message: Some updates to MPPT hardware and software
The design now can charge lead acid batteries but no high/low voltage
cut-out is enabled.
Parts:
- added D3: 1N4004, diode:1N4004
- U$1: value (none) -> 330uF
Connections:
- new net N$1: C6.1, D3.A, R2.1, U$1.P$2
- net EN_: now also EN.1; no longer EN.2
- net GND: no longer EN.1
- net N$12: now also D3.C; no longer C6.1, R2.1, U$1.P$2
- net N$9: now also EN.2
Other:
- note added: "Change Reverse Current Protection"
- moved on the sheet: BATT, EN
Changed lines of the file:
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@@
 <part name="R10" library="rcl" deviceset="R-EU_" device="M0805" value="5"/>
 <part name="C11" library="resistor" deviceset="C-EU" device="C0805K" value="1uF"/>
-<part name="U$1" library="lib" deviceset="INDUC_BOURNES_SDR1806" device=""/>
+<part name="U$1" library="lib" deviceset="INDUC_BOURNES_SDR1806" device="" value="330uF"/>
 <part name="FRAME2" library="frames" deviceset="A3L-LOC" device=""/>
 <part name="SENSE_AMP_SOL" library="equinox" deviceset="ZXCT1107SA-7" device=""/>
@@
 <part name="BATT" library="equinox" deviceset="TERMINAL_2WAY" device=""/>
 <part name="EN" library="jumper" deviceset="SJ" device=""/>
+<part name="D3" library="diode" deviceset="1N4004" device=""/>
 </parts>
 <sheets>
 <sheet>
 <plain>
+<text x="302.26" y="165.1" size="1.778" layer="98">Change Reverse Current Protection</text>
 </plain>
 <instances>
@@
 <instance part="GND3" gate="1" x="297.18" y="200.66"/>
 <instance part="SOL" gate="G$1" x="17.78" y="149.86" rot="MR0"/>
-<instance part="BATT" gate="G$1" x="373.38" y="139.7"/>
-<instance part="EN" gate="1" x="147.32" y="91.44" rot="R90"/>
+<instance part="BATT" gate="G$1" x="370.84" y="139.7"/>
+<instance part="EN" gate="1" x="147.32" y="127" rot="R90"/>
+<instance part="D3" gate="1" x="307.34" y="160.02"/>
 </instances>
 <busses>
@@
 <net name="N$12" class="1">
 <segment>
-<wire x1="293.37" y1="160.02" x2="318.77" y2="160.02" width="0.1524" layer="91"/>
-<wire x1="293.37" y1="172.72" x2="293.37" y2="160.02" width="0.1524" layer="91"/>
-<wire x1="293.37" y1="147.32" x2="293.37" y2="160.02" width="0.1524" layer="91"/>
+<wire x1="309.88" y1="160.02" x2="318.77" y2="160.02" width="0.1524" layer="91"/>
 <wire x1="318.77" y1="125.73" x2="318.77" y2="160.02" width="0.1524" layer="91"/>
-<junction x="293.37" y="160.02"/>
 <pinref part="R5" gate="G$1" pin="2"/>
-<pinref part="R2" gate="G$1" pin="1"/>
-<pinref part="C6" gate="G$1" pin="1"/>
-<pinref part="U$1" gate="G$1" pin="P$2"/>
-<wire x1="292.1" y1="160.02" x2="293.37" y2="160.02" width="0.1524" layer="91"/>
 <pinref part="RSENSE_BATT" gate="G$1" pin="1"/>
 <wire x1="335.28" y1="160.02" x2="340.36" y2="160.02" width="0.1524" layer="91"/>
@@
 <junction x="318.77" y="160.02"/>
 <junction x="335.28" y="160.02"/>
+<pinref part="D3" gate="1" pin="C"/>
 </segment>
 </net>
@@
 <wire x1="177.8" y1="195.58" x2="185.42" y2="195.58" width="0.1524" layer="91"/>
 <wire x1="182.88" y1="116.84" x2="177.8" y2="116.84" width="0.1524" layer="91"/>
-<wire x1="177.8" y1="116.84" x2="177.8" y2="134.62" width="0.1524" layer="91"/>
+<wire x1="177.8" y1="116.84" x2="177.8" y2="132.08" width="0.1524" layer="91"/>
+<wire x1="177.8" y1="132.08" x2="177.8" y2="134.62" width="0.1524" layer="91"/>
 <wire x1="177.8" y1="134.62" x2="187.96" y2="134.62" width="0.1524" layer="91"/>
 <wire x1="177.8" y1="134.62" x2="177.8" y2="195.58" width="0.1524" layer="91"/>
@@
 <wire x1="185.42" y1="195.58" x2="190.5" y2="195.58" width="0.1524" layer="91"/>
 <junction x="185.42" y="195.58"/>
+<pinref part="EN" gate="1" pin="2"/>
+<wire x1="147.32" y1="132.08" x2="177.8" y2="132.08" width="0.1524" layer="91"/>
+<junction x="177.8" y="132.08"/>
 </segment>
 </net>
@@
 <wire x1="137.16" y1="109.22" x2="143.51" y2="109.22" width="0.1524" layer="91"/>
 <label x="144.78" y="109.22" size="1.778" layer="95"/>
-<pinref part="EN" gate="1" pin="2"/>
-<wire x1="147.32" y1="96.52" x2="147.32" y2="106.68" width="0.1524" layer="91"/>
+<pinref part="EN" gate="1" pin="1"/>
+<wire x1="147.32" y1="121.92" x2="147.32" y2="106.68" width="0.1524" layer="91"/>
 <junction x="147.32" y="106.68"/>
 </segment>
@@
 <pinref part="C6" gate="G$1" pin="2"/>
 <wire x1="115.57" y1="78.74" x2="139.7" y2="78.74" width="0.1524" layer="91"/>
-<wire x1="139.7" y1="78.74" x2="147.32" y2="78.74" width="0.1524" layer="91"/>
-<wire x1="147.32" y1="78.74" x2="175.26" y2="78.74" width="0.1524" layer="91"/>
+<wire x1="139.7" y1="78.74" x2="175.26" y2="78.74" width="0.1524" layer="91"/>
 <wire x1="175.26" y1="78.74" x2="243.84" y2="78.74" width="0.1524" layer="91"/>
 <wire x1="243.84" y1="78.74" x2="257.81" y2="78.74" width="0.1524" layer="91"/>
@@
 <wire x1="318.77" y1="100.33" x2="318.77" y2="78.74" width="0.1524" layer="91"/>
 <pinref part="GATE_DRIVE" gate="G$1" pin="COM"/>
-<wire x1="368.3" y1="78.74" x2="345.44" y2="78.74" width="0.1524" layer="91"/>
+<wire x1="365.76" y1="78.74" x2="345.44" y2="78.74" width="0.1524" layer="91"/>
 <junction x="318.77" y="78.74"/>
 <wire x1="345.44" y1="78.74" x2="318.77" y2="78.74" width="0.1524" layer="91"/>
@@
 <wire x1="22.86" y1="147.32" x2="22.86" y2="78.74" width="0.1524" layer="91"/>
 <pinref part="BATT" gate="G$1" pin="P$2"/>
-<wire x1="368.3" y1="78.74" x2="368.3" y2="137.16" width="0.1524" layer="91"/>
+<wire x1="365.76" y1="78.74" x2="365.76" y2="137.16" width="0.1524" layer="91"/>
 <pinref part="U3" gate="A" pin="S"/>
 <pinref part="U3" gate="A" pin="S_3"/>
@@
 <wire x1="243.84" y1="121.92" x2="243.84" y2="78.74" width="0.1524" layer="91"/>
 <junction x="243.84" y="78.74"/>
-<pinref part="EN" gate="1" pin="1"/>
-<wire x1="147.32" y1="86.36" x2="147.32" y2="78.74" width="0.1524" layer="91"/>
-<junction x="147.32" y="78.74"/>
 </segment>
 <segment>
@@
 <junction x="355.6" y="160.02"/>
 <pinref part="BATT" gate="G$1" pin="P$1"/>
-<wire x1="368.3" y1="142.24" x2="368.3" y2="160.02" width="0.1524" layer="91"/>
-<wire x1="368.3" y1="160.02" x2="355.6" y2="160.02" width="0.1524" layer="91"/>
+<wire x1="365.76" y1="142.24" x2="365.76" y2="160.02" width="0.1524" layer="91"/>
+<wire x1="365.76" y1="160.02" x2="355.6" y2="160.02" width="0.1524" layer="91"/>
 </segment>
 </net>
@@
 </segment>
 </net>
+<net name="N$1" class="1">
+<segment>
+<pinref part="D3" gate="1" pin="A"/>
+<wire x1="293.37" y1="160.02" x2="304.8" y2="160.02" width="0.1524" layer="91"/>
+<pinref part="R2" gate="G$1" pin="1"/>
+<wire x1="293.37" y1="172.72" x2="293.37" y2="160.02" width="0.1524" layer="91"/>
+<junction x="293.37" y="160.02"/>
+<pinref part="U$1" gate="G$1" pin="P$2"/>
+<wire x1="292.1" y1="160.02" x2="293.37" y2="160.02" width="0.1524" layer="91"/>
+<wire x1="293.37" y1="147.32" x2="293.37" y2="160.02" width="0.1524" layer="91"/>
+<pinref part="C6" gate="G$1" pin="1"/>
+</segment>
+</net>
