File: Hardware/standalone/standalone.sch (EAGLE design)
At the start: 89 parts, among them Q2 32.768khz, U1 DMS3016SSS-13, U2 DMS3016SSS-13, U3 DMS3016SSS-13, U4 LM2575S-15, U5 NMOS_2N7002, U6 NMOS_2N7002, X1 KUSBVX, X2 KUSBVX

Commit message: Cleaned Library and Complete some ToDo list
Added power LED and changed MPPT reverse current diode
Parts:
- removed D$1: (no value), equinox:DIODE_VS-6CWQ03FN
- removed U$6: 330uF, lib:INDUC_BOURNES_SDR1806
- added D3: (no value), equinox:DIODE_SSB43L
- added LED1: (no value), led:LEDCHIPLED_0805
- added L_MPPT: 330u, equinox:INDUC_BOURNES_SDR1806
- added R21: (no value), resistor:R-EU_M0805
- L_5V: value 330uF -> 330u; device lib:INDUC_BOURNES_SDR1806 -> equinox:INDUC_BOURNES_SDR1806
Connections:
- new net N$37: LED1.C, R21.2
- net +3V3: now also LED1.A
- net GND: now also R21.1
- net N$12: now also D3.ANODE, L_MPPT.P$2; no longer D$1.ANODE_1, D$1.ANODE_2, U$6.P$2
- net N$6: now also L_MPPT.P$1; no longer U$6.P$1
- net V_LOAD: now also D3.CATHODE; no longer D$1.COM_CATHODE
Other:
- note added: "TODO: - Change Caps to surface mount - Battery Bi-Directional Current Sense - Change Current Sense R - Swap 5V Diode to SMT - Check if LCD R/W Pin is needed? - Add filtering (LC) to AVCC - Change Inductors and Cap for Buck - Remove U1 (Not needed) - Change Power Switch - Add serial port"
- note removed: "TODO: - Change Caps to surface mount - Battery Bi-Directional Current Sense - Change Current Sense R - Swap 5V Diode to SMT - Power LED - Check if LCD R/W Pin is needed? - Add filtering (LC) to AVCC - Change Battery Diode to: 1336556 - Change Inductors and Cap for Buck - Remove U1 (Not needed) - Change Power Switch"
Changed lines of the file:
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@@
 <part name="R10" library="rcl" deviceset="R-EU_" device="M0805" value="5"/>
 <part name="C11" library="resistor" deviceset="C-EU" device="C0805K" value="1uF"/>
-<part name="U$6" library="lib" deviceset="INDUC_BOURNES_SDR1806" device="" value="330uF"/>
+<part name="L_MPPT" library="equinox" deviceset="INDUC_BOURNES_SDR1806" device="" value="330u"/>
 <part name="SENSE_AMP_SOL" library="equinox" deviceset="ZXCT1107SA-7" device=""/>
 <part name="R_GAIN" library="rcl" deviceset="R-EU_" device="M0805" value="1k65"/>
@@
 <part name="FRAME3" library="frames" deviceset="A3L-LOC" device=""/>
 <part name="FRAME4" library="frames" deviceset="A3L-LOC" device=""/>
-<part name="D$1" library="equinox" deviceset="DIODE_VS-6CWQ03FN" device=""/>
 <part name="SOL" library="equinox" deviceset="POWER_JACK_2.1MM" device="SLT"/>
 <part name="GND7" library="supply1" deviceset="GND" device=""/>
@@
 <part name="GND18" library="supply1" deviceset="GND" device="" value="GND"/>
 <part name="U4" library="equinox" deviceset="LM2575S-15" device=""/>
-<part name="L_5V" library="lib" deviceset="INDUC_BOURNES_SDR1806" device="" value="330uF"/>
+<part name="L_5V" library="equinox" deviceset="INDUC_BOURNES_SDR1806" device="" value="330u"/>
 <part name="GND19" library="supply1" deviceset="GND" device="" value="GND"/>
 <part name="R11" library="resistor" deviceset="R-EU_" device="M0805" value="75k"/>
@@
 <part name="C19" library="resistor" deviceset="C-EU" device="C0805K" value="1uF"/>
 <part name="C20" library="resistor" deviceset="C-EU" device="C0805K" value="10uF"/>
+<part name="D3" library="equinox" deviceset="DIODE_SSB43L" device=""/>
+<part name="LED1" library="led" deviceset="LED" device="CHIPLED_0805"/>
+<part name="R21" library="resistor" deviceset="R-EU_" device="M0805"/>
+<part name="GND24" library="supply1" deviceset="GND" device=""/>
+<part name="GND25" library="supply1" deviceset="GND" device=""/>
 </parts>
 <sheets>
@@
   - Change Current Sense R
   - Swap 5V Diode to SMT
-  - Power LED
   - Check if LCD R/W Pin is needed?
   - Add filtering (LC) to AVCC
-  - Change Battery Diode to: 1336556
   - Change Inductors and Cap for Buck
   - Remove U1 (Not needed)
-  - Change Power Switch</text>
+  - Change Power Switch
+  - Add serial port</text>
 </plain>
 <instances>
@@
 <instance part="R10" gate="G$1" x="233.68" y="378.46" rot="R270"/>
 <instance part="C11" gate="G$1" x="167.64" y="378.46" rot="R90"/>
-<instance part="U$6" gate="G$1" x="287.02" y="424.18"/>
+<instance part="L_MPPT" gate="1" x="287.02" y="424.18"/>
 <instance part="SENSE_AMP_SOL" gate="A" x="68.58" y="436.88" rot="MR270"/>
 <instance part="R_GAIN" gate="G$1" x="71.12" y="411.48" rot="R90"/>
@@
 <instance part="FRAME3" gate="G$1" x="396.24" y="0"/>
 <instance part="FRAME4" gate="G$1" x="396.24" y="269.24"/>
-<instance part="D$1" gate="G$1" x="307.34" y="424.18"/>
 <instance part="SOL" gate="G$1" x="20.32" y="410.21" smashed="yes">
 <attribute name="VALUE" x="21.59" y="419.1" size="1.778" layer="96" rot="R90"/>
@@
 <instance part="GND18" gate="1" x="279.4" y="185.42"/>
 <instance part="U4" gate="A" x="490.22" y="63.5"/>
-<instance part="L_5V" gate="G$1" x="525.78" y="66.04"/>
+<instance part="L_5V" gate="1" x="525.78" y="66.04"/>
 <instance part="GND19" gate="1" x="467.36" y="33.02"/>
 <instance part="R11" gate="G$1" x="680.72" y="116.84" rot="R90"/>
@@
 <instance part="GND12" gate="1" x="688.34" y="53.34"/>
 <instance part="U$7" gate="A" x="487.68" y="132.08"/>
-<instance part="GND21" gate="1" x="464.82" y="111.76"/>
+<instance part="GND21" gate="1" x="464.82" y="106.68"/>
 <instance part="P+2" gate="1" x="449.58" y="137.16"/>
 <instance part="C17" gate="G$1" x="454.66" y="121.92" rot="R180"/>
 <instance part="C18" gate="G$1" x="518.16" y="121.92" rot="R180"/>
-<instance part="GND22" gate="1" x="518.16" y="111.76"/>
+<instance part="GND22" gate="1" x="518.16" y="106.68"/>
 <instance part="+3V2" gate="G$1" x="520.7" y="137.16" rot="MR0"/>
 <instance part="P+3" gate="1" x="548.64" y="71.12" rot="MR0"/>
@@
 <instance part="C19" gate="G$1" x="86.36" y="408.94" rot="R180"/>
 <instance part="C20" gate="G$1" x="355.6" y="375.92" rot="R180"/>
+<instance part="D3" gate="1" x="304.8" y="424.18"/>
+<instance part="LED1" gate="G$1" x="533.4" y="129.54"/>
+<instance part="R21" gate="G$1" x="533.4" y="116.84" rot="R90"/>
+<instance part="GND24" gate="1" x="533.4" y="106.68"/>
+<instance part="GND25" gate="1" x="454.66" y="106.68"/>
 </instances>
 <busses>
@@
 </segment>
 <segment>
+<pinref part="C17" gate="G$1" pin="1"/>
+<wire x1="454.66" y1="119.38" x2="454.66" y2="109.22" width="0.1524" layer="91"/>
+<pinref part="GND25" gate="1" pin="GND"/>
+</segment>
+<segment>
 <pinref part="U$7" gate="A" pin="GND"/>
 <pinref part="GND21" gate="1" pin="GND"/>
 <wire x1="469.9" y1="127" x2="464.82" y2="127" width="0.1524" layer="91"/>
-<wire x1="464.82" y1="127" x2="464.82" y2="114.3" width="0.1524" layer="91"/>
-<pinref part="C17" gate="G$1" pin="1"/>
-<wire x1="454.66" y1="119.38" x2="454.66" y2="114.3" width="0.1524" layer="91"/>
-<wire x1="454.66" y1="114.3" x2="464.82" y2="114.3" width="0.1524" layer="91"/>
-<junction x="464.82" y="114.3"/>
+<wire x1="464.82" y1="127" x2="464.82" y2="109.22" width="0.1524" layer="91"/>
 </segment>
 <segment>
 <pinref part="GND22" gate="1" pin="GND"/>
 <pinref part="C18" gate="G$1" pin="1"/>
-<wire x1="518.16" y1="114.3" x2="518.16" y2="119.38" width="0.1524" layer="91"/>
+<wire x1="518.16" y1="109.22" x2="518.16" y2="119.38" width="0.1524" layer="91"/>
 </segment>
 <segment>
@@
 <wire x1="116.84" y1="83.82" x2="101.6" y2="83.82" width="0.1524" layer="91"/>
 <junction x="101.6" y="83.82"/>
+</segment>
+<segment>
+<pinref part="R21" gate="G$1" pin="1"/>
+<pinref part="GND24" gate="1" pin="GND"/>
+<wire x1="533.4" y1="109.22" x2="533.4" y2="111.76" width="0.1524" layer="91"/>
 </segment>
 </net>
@@
 <pinref part="C2" gate="G$1" pin="2"/>
 <pinref part="C5" gate="G$1" pin="1"/>
-<pinref part="U$6" gate="G$1" pin="P$1"/>
+<pinref part="L_MPPT" gate="1" pin="P$1"/>
 <wire x1="276.86" y1="424.18" x2="274.32" y2="424.18" width="0.1524" layer="91"/>
 <pinref part="GATE_DRIVE" gate="G$1" pin="VS"/>
@@
 <junction x="325.12" y="424.18"/>
 <label x="332.74" y="441.96" size="1.778" layer="95"/>
-<pinref part="D$1" gate="G$1" pin="COM_CATHODE"/>
-<wire x1="314.96" y1="424.18" x2="318.77" y2="424.18" width="0.1524" layer="91"/>
 <junction x="318.77" y="424.18"/>
+<pinref part="D3" gate="1" pin="CATHODE"/>
+<wire x1="318.77" y1="424.18" x2="309.88" y2="424.18" width="0.1524" layer="91"/>
 </segment>
 <segment>
@@
 <net name="N$12" class="0">
 <segment>
-<pinref part="D$1" gate="G$1" pin="ANODE_1"/>
-<wire x1="302.26" y1="426.72" x2="297.18" y2="426.72" width="0.1524" layer="91"/>
-<wire x1="297.18" y1="426.72" x2="297.18" y2="424.18" width="0.1524" layer="91"/>
-<pinref part="D$1" gate="G$1" pin="ANODE_2"/>
-<wire x1="297.18" y1="424.18" x2="297.18" y2="421.64" width="0.1524" layer="91"/>
-<wire x1="297.18" y1="421.64" x2="302.26" y2="421.64" width="0.1524" layer="91"/>
 <pinref part="R2" gate="G$1" pin="1"/>
 <wire x1="294.64" y1="436.88" x2="294.64" y2="424.18" width="0.1524" layer="91"/>
 <junction x="294.64" y="424.18"/>
-<pinref part="U$6" gate="G$1" pin="P$2"/>
+<pinref part="L_MPPT" gate="1" pin="P$2"/>
 <wire x1="292.1" y1="424.18" x2="294.64" y2="424.18" width="0.1524" layer="91"/>
 <wire x1="294.64" y1="411.48" x2="294.64" y2="424.18" width="0.1524" layer="91"/>
 <pinref part="C6" gate="G$1" pin="1"/>
-<wire x1="297.18" y1="424.18" x2="294.64" y2="424.18" width="0.1524" layer="91"/>
-<junction x="297.18" y="424.18"/>
+<pinref part="D3" gate="1" pin="ANODE"/>
+<wire x1="299.72" y1="424.18" x2="294.64" y2="424.18" width="0.1524" layer="91"/>
 </segment>
 </net>
@@
 <wire x1="518.16" y1="132.08" x2="520.7" y2="132.08" width="0.1524" layer="91"/>
 <wire x1="520.7" y1="132.08" x2="520.7" y2="134.62" width="0.1524" layer="91"/>
+<pinref part="LED1" gate="G$1" pin="A"/>
+<wire x1="520.7" y1="132.08" x2="533.4" y2="132.08" width="0.1524" layer="91"/>
+<junction x="520.7" y="132.08"/>
 </segment>
 <segment>
@@
 <wire x1="508" y1="60.96" x2="535.94" y2="60.96" width="0.1524" layer="91"/>
 <wire x1="535.94" y1="60.96" x2="535.94" y2="66.04" width="0.1524" layer="91"/>
-<pinref part="L_5V" gate="G$1" pin="P$2"/>
+<pinref part="L_5V" gate="1" pin="P$2"/>
 <wire x1="535.94" y1="66.04" x2="530.86" y2="66.04" width="0.1524" layer="91"/>
 <wire x1="535.94" y1="66.04" x2="541.02" y2="66.04" width="0.1524" layer="91"/>
@@
 <net name="N$21" class="0">
 <segment>
-<pinref part="L_5V" gate="G$1" pin="P$1"/>
+<pinref part="L_5V" gate="1" pin="P$1"/>
 <pinref part="U4" gate="A" pin="OUT"/>
 <wire x1="515.62" y1="66.04" x2="513.08" y2="66.04" width="0.1524" layer="91"/>
@@
 </segment>
 </net>
+<net name="N$37" class="0">
+<segment>
+<pinref part="LED1" gate="G$1" pin="C"/>
+<pinref part="R21" gate="G$1" pin="2"/>
+<wire x1="533.4" y1="124.46" x2="533.4" y2="121.92" width="0.1524" layer="91"/>
+</segment>
+</net>

Commit message: Many PCB Improvements
Tidied up Silkscreen.
Changed some through hole components to surface mount.
Changed the 15V regulator for 5V as originally intended.
Checked power rating of converters. Need to update 5V out to 3A.
On PCB, tidied up the 12V track and thickened so that it can carry
larger current.
Parts:
- removed D5: (no value), diode:ZENER-DIODEDO41Z10
- removed U$5: STM32F050C6T6A, equinox:STM32F050C6T6A
- added D6: B340-13-F, equinox:DIODE_B340-13-F
- added IC1: STM32F050C6T6A, equinox:STM32F050C6T6A
- added SERIAL: (no value), pinhead:PINHD-1X3
- 5V_CIN: device capacitor-wima:C2.5/2 -> resistor:CPOL-EUE
- 5V_COUT: device capacitor-wima:C2.5/2 -> resistor:CPOL-EUF
- C4: device resistor:C-EU025-050X050 -> resistor:CPOL-EUE
- C6: device resistor:C-EU025-050X050 -> resistor:CPOL-EUF
- LED1: value (none) -> POW_3V3
- R21: value (none) -> 1K
- U4: value LM2575S-15 -> LM2575S-5; device equinox:LM2575S-15 -> equinox:LM2575S-5
- renumbered U$7 to VREG, U$8 to IC2
Connections:
- net +3V3: now also IC1.VDD, IC1.VDDA, IC1.VDD_; no longer U$5.VDD, U$5.VDDA, U$5.VDD_
- net +5V: now also 5V_COUT.+; no longer 5V_COUT.1
- net 12V_OUT_EN: now also IC1.PA12; no longer U$5.PA12
- net BATT_I: now also IC1.PA4; no longer U$5.PA4
- net BATT_V: now also IC1.PA3; no longer U$5.PA3
- net CC_PWM: now also IC1.PA7; no longer U$5.PA7
- net CC_~EN: now also IC1.PB0; no longer U$5.PB0
- net GND: now also 5V_CIN.-, 5V_COUT.-, C4.-, C6.-, D6.ANODE, IC1.BOOT0, IC1.VSS, IC1.VSSA, IC1.VSS_, SERIAL.3; no longer 5V_CIN.2, 5V_COUT.2, C4.2, C6.2, D5.A, U$5.BOOT0, U$5.VSS, U$5.VSSA, U$5.VSS_
- net LCD_BK_EN: now also IC1.PB1; no longer U$5.PB1
- net LCD_D4: now also IC1.PB15; no longer U$5.PB15
- net LCD_D5: now also IC1.PB14; no longer U$5.PB14
- net LCD_D6: now also IC1.PB13; no longer U$5.PB13
- net LCD_D7: now also IC1.PB12; no longer U$5.PB12
- net LCD_E: now also IC1.PB11; no longer U$5.PB11
- net LCD_RS: now also IC1.PB2; no longer U$5.PB2
- net LCD_RW: now also IC1.PB10; no longer U$5.PB10
- net N$1: now also IC1.PC14_OSC32_IN; no longer U$5.PC14_OSC32_IN
- net N$12: now also C6.+; no longer C6.1
- net N$18: now also IC1.PC15_OSC32_OUT; no longer U$5.PC15_OSC32_OUT
- net N$21: now also D6.CATHODE; no longer D5.C
- net N$22: now also IC1.PA8; no longer U$5.PA8
- net N$23: now also IC1.PB9; no longer U$5.PB9
- net N$24: now also IC1.PB8; no longer U$5.PB8
- net N$26: now also IC1.PB7; no longer U$5.PB7
- net N$27: now also IC1.PB6; no longer U$5.PB6
- net N$28: now also IC1.PB5; no longer U$5.PB5
- net N$29: now also IC1.PB4; no longer U$5.PB4
- net N$30: now also IC1.PA15; no longer U$5.PA15
- net N$9: now also C4.+; no longer C4.1
- net NRST: now also IC1.NRST; no longer U$5.NRST
- net SOL_I: now also IC1.PA2; no longer U$5.PA2
- net SOL_V: now also IC1.PA1; no longer U$5.PA1
- net SWCLK: now also IC1.PA14; no longer U$5.PA14
- net SWDIO: now also IC1.PA13; no longer U$5.PA13
- net SWO: now also IC1.PB3; no longer U$5.PB3
- net USART1_RX: now also IC1.PA10, SERIAL.1; no longer U$5.PA10
- net USART1_TX: now also IC1.PA9, SERIAL.2; no longer U$5.PA9
- net USB_EN1: now also IC1.PF7; no longer U$5.PF7
- net USB_EN2: now also IC1.PF6; no longer U$5.PF6
- net USB_FLG1: now also IC1.PA5; no longer U$5.PA5
- net USB_FLG2: now also IC1.PA6; no longer U$5.PA6
- net V_BACKUP: now also IC1.VBATT; no longer U$5.VBATT
- net V_LOAD: now also 5V_CIN.+; no longer 5V_CIN.1
- net WKUP: now also IC1.PA0; no longer U$5.PA0
Other:
- note added: "120mA Max"
- note added: "1A Current Limit"
- note added: "1A Output"
- note added: "250mA Output"
- note added: "Must be 0placed near to IC1"
- note added: "Replace"
- note added: "Replace with LM2576"
- note added: "Replace with: 1612709"
- note added: "TODO: - Battery Bi-Directional Current Sense - Change Current Sense R - Check if LCD R/W Pin is needed? - Add filtering (LC) to AVCC - Change Inductors and Cap for Buck - Remove U1 (Not needed) - Change Power Switch - Place Keep-out border around the edge of board - Contrast Adjust Pot needs changing - Swap LM2575 with LM2576 and change L/C"
- note removed: "TODO: - Change Caps to surface mount - Battery Bi-Directional Current Sense - Change Current Sense R - Swap 5V Diode to SMT - Check if LCD R/W Pin is needed? - Add filtering (LC) to AVCC - Change Inductors and Cap for Buck - Remove U1 (Not needed) - Change Power Switch - Add serial port"
- moved on the sheet: LED1
