File: Hardware/standalone/standalone.sch (EAGLE design)
At the start: 92 parts, among them IC1 STM32F050C6T6A, IC2 AP1212, Q2 32.768khz, U1 DMS3016SSS-13, U2 DMS3016SSS-13, U3 DMS3016SSS-13, U4 LM2575S-5, U5 NMOS_2N7002, U6 NMOS_2N7002, X1 KUSBVX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

Commit message: Increase 5V Output to 3A max
Switched SMPS Controller, Inductor and Capacitor.
Parts:
- 5V_COUT: value 330u -> 1000uF; device resistor:CPOL-EUF -> resistor:CPOL-EUG
- L_5V: value 330u -> 100uH; device equinox:INDUC_BOURNES_SDR1806 -> equinox:INDUC_BOURNES_SDR2207
- SOL: value POWER_JACK_2.1MMSLT -> (none); device equinox:POWER_JACK_2.1MMSLT -> con-jack:JACK-PLUG0
- U4: value LM2575S-5 -> LM2576S; device equinox:LM2575S-5 -> equinox:LM2576S
Connections:
- net GND: now also SOL.1, SOL.2; no longer SOL.GND, SOL.GNDBREAK
- net N$16: now also SOL.3; no longer SOL.PWR
Other:
- note added: "3A Output"
- note added: "TODO: - Battery Bi-Directional Current Sense - Change Current Sense R - Check if LCD R/W Pin is needed? - Add filtering (LC) to AVCC - Change Inductors and Cap for Buck - Remove U1 (Not needed) - Change Power Switch - Place Keep-out border around the edge of board - Contrast Adjust Pot needs changing"
- note removed: "1A Output"
- note removed: "Replace"
- note removed: "Replace with LM2576"
- note removed: "Replace with: 1612709"
- note removed: "TODO: - Battery Bi-Directional Current Sense - Change Current Sense R - Check if LCD R/W Pin is needed? - Add filtering (LC) to AVCC - Change Inductors and Cap for Buck - Remove U1 (Not needed) - Change Power Switch - Place Keep-out border around the edge of board - Contrast Adjust Pot needs changing - Swap LM2575 with LM2576 and change L/C"
Changed lines of the file:
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@@
 <part name="FRAME3" library="frames" deviceset="A3L-LOC" device=""/>
 <part name="FRAME4" library="frames" deviceset="A3L-LOC" device=""/>
-<part name="SOL" library="equinox" deviceset="POWER_JACK_2.1MM" device="SLT"/>
 <part name="GND7" library="supply1" deviceset="GND" device=""/>
 <part name="BATT_BCKUP" library="coin_cells" deviceset="PANASONIC_CR2032_1298246" device="" value="RENATA_COIN_CELL"/>
@@
 <part name="+3V7" library="supply1" deviceset="+3V3" device=""/>
 <part name="GND18" library="supply1" deviceset="GND" device="" value="GND"/>
-<part name="L_5V" library="equinox" deviceset="INDUC_BOURNES_SDR1806" device="" value="330u"/>
+<part name="L_5V" library="equinox" deviceset="INDUC_BOURNES_SDR2207" device="" value="100uH"/>
 <part name="GND19" library="supply1" deviceset="GND" device="" value="GND"/>
 <part name="R11" library="resistor" deviceset="R-EU_" device="M0805" value="75k"/>
@@
 <part name="+3V2" library="supply1" deviceset="+3V3" device=""/>
 <part name="P+3" library="supply1" deviceset="+5V" device=""/>
-<part name="5V_COUT" library="resistor" deviceset="CPOL-EU" device="F" value="330u"/>
+<part name="5V_COUT" library="resistor" deviceset="CPOL-EU" device="G" value="1000uF"/>
 <part name="5V_CIN" library="resistor" deviceset="CPOL-EU" device="E" value="100u"/>
 <part name="IC2" library="equinox" deviceset="AP1212" device=""/>
@@
 <part name="SERIAL" library="pinhead" deviceset="PINHD-1X3" device=""/>
 <part name="GND26" library="supply1" deviceset="GND" device="" value="GND"/>
-<part name="U4" library="equinox" deviceset="LM2575S-5" device=""/>
+<part name="U4" library="equinox" deviceset="LM2576S" device=""/>
 <part name="D6" library="equinox" deviceset="DIODE_B340-13-F" device="" value="B340-13-F"/>
 <part name="GND27" library="supply1" deviceset="GND" device="" value="GND"/>
 <part name="GND28" library="supply1" deviceset="GND" device="" value="GND"/>
 <part name="GND29" library="supply1" deviceset="GND" device="" value="GND"/>
+<part name="SOL" library="con-jack" deviceset="JACK-PLUG" device="0"/>
 </parts>
 <sheets>
@@
   - Change Power Switch
   - Place Keep-out border around the edge of board
-  - Contrast Adjust Pot needs changing
-  - Swap LM2575 with LM2576 and change L/C</text>
+  - Contrast Adjust Pot needs changing</text>
 <text x="662.94" y="127" size="1.778" layer="98">1A Current Limit</text>
 <text x="662.94" y="86.36" size="1.778" layer="98">1A Current Limit</text>
-<text x="510.54" y="73.66" size="1.778" layer="98">Replace with: 1612709</text>
-<text x="551.18" y="40.64" size="1.778" layer="98" rot="R90">Replace</text>
-<text x="480.06" y="43.18" size="1.778" layer="98">Replace with LM2576</text>
-<text x="556.26" y="66.04" size="1.778" layer="98" rot="R90">1A Output</text>
+<text x="556.26" y="66.04" size="1.778" layer="98" rot="R90">3A Output</text>
 <text x="208.28" y="88.9" size="1.778" layer="98">120mA Max</text>
 <text x="556.26" y="132.08" size="1.778" layer="98" rot="R90">250mA Output</text>
@@
 <instance part="FRAME3" gate="G$1" x="396.24" y="0"/>
 <instance part="FRAME4" gate="G$1" x="396.24" y="269.24"/>
-<instance part="SOL" gate="G$1" x="20.32" y="410.21" smashed="yes">
-<attribute name="VALUE" x="21.59" y="419.1" size="1.778" layer="96" rot="R90"/>
-<attribute name="NAME" x="10.16" y="410.21" size="1.778" layer="95"/>
-</instance>
 <instance part="GND7" gate="1" x="487.68" y="175.26"/>
 <instance part="BATT_BCKUP" gate="G$1" x="487.68" y="190.5"/>
@@
 <instance part="SERIAL" gate="A" x="30.48" y="193.04" rot="MR0"/>
 <instance part="GND26" gate="1" x="66.04" y="182.88"/>
-<instance part="U4" gate="A" x="490.22" y="63.5"/>
+<instance part="U4" gate="1" x="490.22" y="60.96"/>
 <instance part="D6" gate="1" x="513.08" y="50.8" rot="R90"/>
 <instance part="GND27" gate="1" x="513.08" y="33.02"/>
 <instance part="GND28" gate="1" x="541.02" y="33.02"/>
 <instance part="GND29" gate="1" x="436.88" y="33.02"/>
+<instance part="SOL" gate="G$1" x="17.78" y="411.48"/>
 </instances>
 <busses>
@@
 <wire x1="68.58" y1="452.12" x2="59.69" y2="459.74" width="0.1524" layer="91"/>
 <junction x="59.69" y="459.74"/>
-<wire x1="22.86" y1="417.83" x2="22.86" y2="459.74" width="0.1524" layer="91"/>
-<pinref part="SOL" gate="G$1" pin="PWR"/>
+<pinref part="SOL" gate="G$1" pin="3"/>
+<wire x1="22.86" y1="414.02" x2="22.86" y2="459.74" width="0.1524" layer="91"/>
 </segment>
 </net>
@@
 <wire x1="345.44" y1="342.9" x2="345.44" y2="372.11" width="0.1524" layer="91"/>
 <junction x="345.44" y="342.9"/>
-<wire x1="22.86" y1="412.75" x2="22.86" y2="342.9" width="0.1524" layer="91"/>
+<wire x1="22.86" y1="408.94" x2="22.86" y2="342.9" width="0.1524" layer="91"/>
 <wire x1="365.76" y1="342.9" x2="365.76" y2="398.78" width="0.1524" layer="91"/>
 <pinref part="U3" gate="A" pin="S"/>
@@
 <junction x="243.84" y="342.9"/>
 <pinref part="BATT" gate="CON$2" pin="S"/>
-<pinref part="SOL" gate="G$1" pin="GND"/>
-<wire x1="22.86" y1="415.29" x2="22.86" y2="412.75" width="0.1524" layer="91"/>
-<junction x="22.86" y="412.75"/>
-<pinref part="SOL" gate="G$1" pin="GNDBREAK"/>
 <pinref part="R_GAIN" gate="G$1" pin="1"/>
 <wire x1="71.12" y1="406.4" x2="71.12" y2="342.9" width="0.1524" layer="91"/>
@@
 <wire x1="355.6" y1="373.38" x2="355.6" y2="342.9" width="0.1524" layer="91"/>
 <junction x="355.6" y="342.9"/>
+<pinref part="SOL" gate="G$1" pin="2"/>
+<wire x1="22.86" y1="411.48" x2="22.86" y2="408.94" width="0.1524" layer="91"/>
+<pinref part="SOL" gate="G$1" pin="1"/>
+<junction x="22.86" y="408.94"/>
 </segment>
 <segment>
@@
 <segment>
 <pinref part="GND19" gate="1" pin="GND"/>
-<pinref part="U4" gate="A" pin="GND_2"/>
+<pinref part="U4" gate="1" pin="GND_2"/>
 <wire x1="472.44" y1="55.88" x2="467.36" y2="55.88" width="0.1524" layer="91"/>
-<pinref part="U4" gate="A" pin="~ON~/OFF"/>
+<pinref part="U4" gate="1" pin="~ON~/OFF"/>
 <wire x1="472.44" y1="60.96" x2="467.36" y2="60.96" width="0.1524" layer="91"/>
 <wire x1="467.36" y1="60.96" x2="467.36" y2="55.88" width="0.1524" layer="91"/>
@@
 <wire x1="467.36" y1="55.88" x2="467.36" y2="53.34" width="0.1524" layer="91"/>
 <wire x1="467.36" y1="53.34" x2="467.36" y2="35.56" width="0.1524" layer="91"/>
-<pinref part="U4" gate="A" pin="GND"/>
+<pinref part="U4" gate="1" pin="GND"/>
 <wire x1="472.44" y1="53.34" x2="467.36" y2="53.34" width="0.1524" layer="91"/>
 <junction x="467.36" y="53.34"/>
@@
 <junction x="436.88" y="66.04"/>
 <label x="424.18" y="66.04" size="1.778" layer="95"/>
-<pinref part="U4" gate="A" pin="VIN"/>
+<pinref part="U4" gate="1" pin="VIN"/>
 </segment>
 </net>
@@
 <wire x1="548.64" y1="68.58" x2="548.64" y2="66.04" width="0.1524" layer="91"/>
 <wire x1="548.64" y1="66.04" x2="541.02" y2="66.04" width="0.1524" layer="91"/>
-<pinref part="U4" gate="A" pin="FB"/>
+<pinref part="U4" gate="1" pin="FB"/>
 </segment>
 <segment>
@@
 <wire x1="513.08" y1="66.04" x2="508" y2="66.04" width="0.1524" layer="91"/>
 <junction x="513.08" y="66.04"/>
-<pinref part="U4" gate="A" pin="OUT"/>
+<pinref part="U4" gate="1" pin="OUT"/>
 <pinref part="D6" gate="1" pin="CATHODE"/>
 <wire x1="513.08" y1="55.88" x2="513.08" y2="66.04" width="0.1524" layer="91"/>
