File: Hardware/standalone/standalone.sch (EAGLE design)
At the start: 91 parts, among them IC1 STM32F050C6T6A, IC2 AP1212, Q2 32.768khz, U1 NMOS_2N7002, U10 ZXCT1107SA-7, U2 FDS6690a, U3 FDS6690a, U4 LM2576S, U5 NMOS_2N7002, U6 NMOS_2N7002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

Commit message: Hardware fixes
Parts:
- removed C16: 1uF, resistor:C-EUC0805K
- added R29: 1k, resistor:R-EU_M0805
- added U8: NMOS_2N7002, equinox:NMOS_2N7002
- POW: RS (none) -> 758-1979
- R4, R6: value 1.32k -> 1.33k
Connections:
- new net N$42: BUZZ1.-, U8.D
- new net N$43: R29.2, U8.G
- net GND: now also U8.S; no longer BUZZ1.-, C16.1
- net N$22: now also R29.1; no longer BUZZ1.+
- net V_BACKUP: no longer C16.2
- net V_LOAD: now also BUZZ1.+
Other:
- note added: "Must be placed near to IC1"
- note added: "TODO: - Contrast Adjust Pot needs changing - Add PTC & Diode"
- note removed: "Must be 0placed near to IC1"
- note removed: "TODO: - Contrast Adjust Pot needs changing - Add PTC & Diode - Change Buzzer and add mosfet switching for higher voltage, thus louder"
Changed lines of the file:
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@@
 </part>
 <part name="R3" library="rcl" deviceset="R-EU_" device="M0805" value="10K"/>
-<part name="R4" library="rcl" deviceset="R-EU_" device="M0805" value="1.32k"/>
+<part name="R4" library="rcl" deviceset="R-EU_" device="M0805" value="1.33k"/>
 <part name="C7" library="resistor" deviceset="C-EU" device="C0805K" value="10uF"/>
 <part name="R5" library="rcl" deviceset="R-EU_" device="M0805" value="10K"/>
-<part name="R6" library="rcl" deviceset="R-EU_" device="M0805" value="1.32k"/>
+<part name="R6" library="rcl" deviceset="R-EU_" device="M0805" value="1.33k"/>
 <part name="C8" library="resistor" deviceset="C-EU" device="C0805K" value="10uF"/>
 <part name="R8" library="rcl" deviceset="R-EU_" device="M0805" value="200"/>
@@
 <part name="C14" library="resistor" deviceset="C-EU" device="C0805K" value="100nF"/>
 <part name="C15" library="resistor" deviceset="C-EU" device="C0805K" value="100nF"/>
-<part name="C16" library="resistor" deviceset="C-EU" device="C0805K" value="1uF"/>
 <part name="P+1" library="supply1" deviceset="+5V" device=""/>
 <part name="GND17" library="supply1" deviceset="GND" device="" value="GND"/>
@@
 <part name="+3V8" library="supply1" deviceset="+3V3" device=""/>
 <part name="GND23" library="supply1" deviceset="GND" device="" value="GND"/>
-<part name="POW" library="equinox" deviceset="TAC_SWITCH" device="PTH"/>
+<part name="POW" library="equinox" deviceset="TAC_SWITCH" device="PTH">
+<attribute name="RS" value="758-1979"/>
+</part>
 <part name="R24" library="resistor" deviceset="R-EU_" device="M0805" value="1k"/>
 <part name="GND3" library="supply1" deviceset="GND" device="" value="GND"/>
@@
 <part name="R28" library="rcl" deviceset="R-EU_" device="M0805" value="10"/>
 <part name="C20" library="resistor" deviceset="C-EU" device="C0805K" value="10uF"/>
+<part name="U8" library="equinox" deviceset="NMOS_2N7002" device="">
+<attribute name="MPN" value="2N7002-7-F"/>
+<attribute name="OC_FARNELL" value="1713823"/>
+<attribute name="OC_NEWARK" value="25R5679"/>
+<attribute name="PACKAGE" value="SOT-23-3"/>
+<attribute name="SUPPLIER" value="DIODES INC."/>
+</part>
+<part name="R29" library="resistor" deviceset="R-EU_" device="M0805" value="1k"/>
 </parts>
 <sheets>
@@
   - Contrast Adjust Pot needs changing
   - Add PTC &amp; Diode
-  - Change Buzzer and add mosfet switching for higher voltage, thus louder
 </text>
 <text x="662.94" y="127" size="1.778" layer="98">0.5A Current Limit</text>
@@
 <text x="208.28" y="88.9" size="1.778" layer="98">120mA Max</text>
 <text x="556.26" y="132.08" size="1.778" layer="98" rot="R90">250mA Output</text>
-<text x="297.18" y="66.04" size="1.778" layer="98">Must be 0placed near to IC1</text>
+<text x="297.18" y="66.04" size="1.778" layer="98">Must be placed near to IC1</text>
 <text x="355.6" y="426.72" size="1.778" layer="98">Add PTC: 1800724
 And Diode</text>
@@
 <instance part="C14" gate="G$1" x="322.58" y="50.8" rot="R180"/>
 <instance part="C15" gate="G$1" x="332.74" y="50.8" rot="R180"/>
-<instance part="C16" gate="G$1" x="477.52" y="190.5" rot="R180"/>
 <instance part="P+1" gate="1" x="279.4" y="226.06"/>
-<instance part="GND17" gate="1" x="259.08" y="99.06"/>
+<instance part="GND17" gate="1" x="259.08" y="66.04"/>
 <instance part="KEYPAD" gate="A" x="193.04" y="231.14" rot="R90">
 <attribute name="OC_FARNELL" x="193.04" y="231.14" size="1.778" layer="96" rot="R90" display="off"/>
@@
 <instance part="+3V8" gate="G$1" x="63.5" y="228.6"/>
 <instance part="GND23" gate="1" x="68.58" y="205.74"/>
-<instance part="POW" gate="S" x="101.6" y="109.22" rot="R90"/>
+<instance part="POW" gate="S" x="101.6" y="109.22" rot="R90">
+<attribute name="RS" x="101.6" y="109.22" size="1.778" layer="96" rot="R90" display="off"/>
+</instance>
 <instance part="R24" gate="G$1" x="101.6" y="91.44" rot="R270"/>
 <instance part="GND3" gate="1" x="101.6" y="78.74"/>
@@
 <instance part="R28" gate="G$1" x="337.82" y="414.02" rot="R90"/>
 <instance part="C20" gate="G$1" x="334.01" y="407.67" rot="R270"/>
+<instance part="U8" gate="A" x="256.54" y="83.82"/>
+<instance part="R29" gate="G$1" x="248.92" y="96.52" rot="R270"/>
 </instances>
 <busses>
@@
 <pinref part="U4" gate="1" pin="VIN"/>
 </segment>
+<segment>
+<pinref part="BUZZ1" gate="G$1" pin="+"/>
+<wire x1="259.08" y1="114.3" x2="259.08" y2="129.54" width="0.1524" layer="91"/>
+<wire x1="259.08" y1="129.54" x2="276.86" y2="129.54" width="0.1524" layer="91"/>
+<label x="264.16" y="129.54" size="1.778" layer="95"/>
+</segment>
 </net>
 <net name="N$12" class="0">
@@
 <wire x1="487.68" y1="205.74" x2="508" y2="205.74" width="0.1524" layer="91"/>
 <label x="492.76" y="205.74" size="1.778" layer="95"/>
-<pinref part="C16" gate="G$1" pin="2"/>
-<wire x1="477.52" y1="195.58" x2="477.52" y2="205.74" width="0.1524" layer="91"/>
-<wire x1="477.52" y1="205.74" x2="487.68" y2="205.74" width="0.1524" layer="91"/>
-<junction x="487.68" y="205.74"/>
 </segment>
 </net>
@@
 <segment>
 <pinref part="IC1" gate="1" pin="PA8"/>
-<pinref part="BUZZ1" gate="G$1" pin="+"/>
-<wire x1="259.08" y1="114.3" x2="259.08" y2="119.38" width="0.1524" layer="91"/>
-<wire x1="259.08" y1="119.38" x2="220.98" y2="119.38" width="0.1524" layer="91"/>
+<wire x1="248.92" y1="119.38" x2="220.98" y2="119.38" width="0.1524" layer="91"/>
+<pinref part="R29" gate="G$1" pin="1"/>
+<wire x1="248.92" y1="101.6" x2="248.92" y2="119.38" width="0.1524" layer="91"/>
 </segment>
 </net>
@@
 </net>
 <net name="GND" class="1">
-<segment>
-<pinref part="BUZZ1" gate="G$1" pin="-"/>
-<pinref part="GND17" gate="1" pin="GND"/>
-<wire x1="259.08" y1="106.68" x2="259.08" y2="101.6" width="0.1524" layer="91"/>
-</segment>
 <segment>
 <wire x1="115.57" y1="336.55" x2="115.57" y2="342.9" width="0.1524" layer="91"/>
@@
 </segment>
 <segment>
+<pinref part="BATT_BCKUP" gate="G$1" pin="NEG"/>
 <wire x1="487.68" y1="180.34" x2="487.68" y2="177.8" width="0.1524" layer="91"/>
 <pinref part="GND7" gate="1" pin="GND"/>
-<pinref part="BATT_BCKUP" gate="G$1" pin="NEG"/>
-<pinref part="C16" gate="G$1" pin="1"/>
-<wire x1="477.52" y1="187.96" x2="477.52" y2="180.34" width="0.1524" layer="91"/>
-<wire x1="477.52" y1="180.34" x2="487.68" y2="180.34" width="0.1524" layer="91"/>
-<junction x="487.68" y="180.34"/>
 </segment>
 <segment>
@@
 <pinref part="U1" gate="A" pin="S"/>
 <wire x1="289.56" y1="165.1" x2="289.56" y2="167.64" width="0.1524" layer="91"/>
+</segment>
+<segment>
+<pinref part="GND17" gate="1" pin="GND"/>
+<pinref part="U8" gate="A" pin="S"/>
+<wire x1="259.08" y1="68.58" x2="259.08" y2="73.66" width="0.1524" layer="91"/>
 </segment>
 </net>
@@
 </segment>
 </net>
+<net name="N$42" class="0">
+<segment>
+<pinref part="U8" gate="A" pin="D"/>
+<pinref part="BUZZ1" gate="G$1" pin="-"/>
+<wire x1="259.08" y1="91.44" x2="259.08" y2="106.68" width="0.1524" layer="91"/>
+</segment>
+</net>
+<net name="N$43" class="0">
+<segment>
+<pinref part="R29" gate="G$1" pin="2"/>
+<pinref part="U8" gate="A" pin="G"/>
+<wire x1="248.92" y1="78.74" x2="248.92" y2="91.44" width="0.1524" layer="91"/>
+</segment>
+</net>
