File: Hardware/standalone_pro/standalone.sch (EAGLE design)
At the start: 112 parts, among them IC1 IR2104S, IC2 STM32F050C6T6A, IC3 AP1212, IC4 AP1212, Q1 32.768kHz, U1 ZXCT1107SA-7, U10 NMOS_2N7002, U2 NMOS_2N7002, U3 NMOS_2N7002, U4 FDS6690a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

Commit message: Pro hardware ready for first prototype
Parts:
- removed PTC1: 7A, equinox:PTC_MF_R700
Connections:
- removed net N$46: BATTCON$1.S, PTC1.P$2
- net N$4: now also BATTCON$1.S; no longer PTC1.P$1
Changed lines of the file:
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@@
 <part name="+3V11" library="supply1" deviceset="+3V3" device=""/>
 <part name="GND31" library="supply1" deviceset="GND" device="" value="GND"/>
-<part name="PTC1" library="equinox" deviceset="PTC_MF_R700" device="" value="7A"/>
 <part name="D5" library="equinox" deviceset="DIODE_SSB43L" device="" value="SSB43L">
 <attribute name="OC_FARNELL" value="1336556"/>
@@
 <instance part="+3V11" gate="G$1" x="121.92" y="119.38"/>
 <instance part="GND31" gate="1" x="114.3" y="30.48"/>
-<instance part="PTC1" gate="PTC1" x="363.22" y="424.18"/>
 <instance part="D5" gate="1" x="358.14" y="398.78" rot="R90">
 <attribute name="OC_FARNELL" x="358.14" y="398.78" size="1.778" layer="96" rot="R90" display="off"/>
@@
 <wire x1="358.14" y1="424.18" x2="332.74" y2="424.18" width="0.1524" layer="91"/>
 <wire x1="327.66" y1="419.1" x2="332.74" y2="424.18" width="0.1524" layer="91"/>
-<pinref part="PTC1" gate="PTC1" pin="P$1"/>
 <pinref part="D5" gate="1" pin="CATHODE"/>
 <wire x1="358.14" y1="403.86" x2="358.14" y2="424.18" width="0.1524" layer="91"/>
+<wire x1="373.38" y1="403.86" x2="373.38" y2="424.18" width="0.1524" layer="91"/>
+<pinref part="BATT" gate="CON$1" pin="S"/>
+<wire x1="358.14" y1="424.18" x2="373.38" y2="424.18" width="0.1524" layer="91"/>
 <junction x="358.14" y="424.18"/>
 </segment>
@@
 </segment>
 </net>
-<net name="N$46" class="1">
-<segment>
-<pinref part="PTC1" gate="PTC1" pin="P$2"/>
-<wire x1="373.38" y1="424.18" x2="370.84" y2="424.18" width="0.1524" layer="91"/>
-<wire x1="373.38" y1="403.86" x2="373.38" y2="424.18" width="0.1524" layer="91"/>
-<pinref part="BATT" gate="CON$1" pin="S"/>
-</segment>
-</net>

Commit message: Updates Pro MPPT Inductor Part #
Parts:
- L_MPPT: OC_FARNELL 1929706 -> 1077018
Changed lines of the file:
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@@
 <part name="C9" library="resistor" deviceset="C-EU" device="C0805K" value="1uF"/>
 <part name="L_MPPT" library="equinox" deviceset="INDUC_MURATA_1433428C" device="" value="330u">
-<attribute name="OC_FARNELL" value="1929706"/>
+<attribute name="OC_FARNELL" value="1077018"/>
 </part>
 <part name="U1" library="equinox" deviceset="ZXCT1107SA-7" device=""/>
